File: KiCad/VCO_RPIpico.kicad_sch (KiCad schematic)
At the start: 81 parts, among them J1 AudioJack3_Ground, J2 Power Jack, SW1 LFO1/2, SW2 Select LFO WaveForm, SW3 Fire4, SW4 Fire3, SW5 Fire2, SW6 Fire1, SW7 Shift2/Save, SW8 Shift1 / Select Bank, U2 PT2399, U3 L7805

Commit message: Kicad: Muting control added
Parts:
- added C25: 1µ, Capacitor_Tantalum_SMD:CP_EIA-2012-12_Kemet-R_Pad1.30x1.05mm_HandSolder, symbol Device:C_Polarized
- added Q1: 2N7002, Package_TO_SOT_SMD:SOT-23, symbol Transistor_FET:2N7002
- added R31: 10k, Resistor_SMD:R_1206_3216Metric, symbol Device:R
Connections:
- net GND: now also C25.2, Q1.2 (S)
- net Wave_out: now also Q1.3 (D)
- net mute: now reaches A1.29 (GPIO22)
- net mute: now also R31.2
- new net: C25.1, Q1.1 (G), R31.1
- no-connect marks 11 -> 10
Other:
- note added: "a)"
