File: KiCad/VCO_RPIpico.kicad_pcb (KiCad board)
At the start: 2 copper layers, 142 x 67 mm, 48 parts, among them J1 AudioJack2, J2 Power Jack 5V, J3 Wave Out, J4 Echo Out, J5 Poti Echo Mix/Feedback, J6 Poti Echo Freq, J7 Echo Power, Q1 PNP, SW1 Select Waveform, SW3 Fire4, SW4 Fire3, SW5 Fire2, SW6 Fire1, SW7 Shift2/Save, SW8 Shift1

Commit message: Kicad
Parts:
- removed D8: LED_Shift2, LED_THT:LED_D3.0mm-3
- removed Q1: PNP, Package_TO_SOT_SMD:SOT-23
- removed R16: 1k, Resistor_SMD:R_1206_3216Metric
- added D3: LED Shift1, LED_THT:LED_D3.0mm, F.Cu at (157.3, 87.0)
- added D9: LED Shift2, LED_THT:LED_D3.0mm, F.Cu at (175.4, 87.0)
- added R17: 100, Resistor_SMD:R_1206_3216Metric, B.Cu at (135.5, 82.5)
- added SW2: Select Waveform LFO2, Button_Switch_THT:SW_PUSH_6mm, F.Cu at (141.2, 96.2)
- SW1: value Select Waveform -> Select Waveform LFO1
- SW8: value Shift1 -> Shift1 / Select Bank
- moved R7 12.7 mm to (154.8, 82.5)
- moved R8 10.2 mm to (172.8, 82.5)
- moved D1 9.00 mm to (140.5, 87.0)
- moved SW1 9.00 mm to (123.2, 96.2)
- moved SW7 9.00 mm to (177.2, 96.2)
- moved SW8 9.00 mm to (159.2, 96.2)
- moved D2 9.00 mm to (122.5, 87.0)
Connections:
- A1 pad 19: unconnected-(A1-GPIO14-Pad19)_1 -> Net-(A1-GPIO14)
- A1 pad 20: unconnected-(A1-GPIO15-Pad20)_1 -> Net-(A1-GPIO15)
- A1 pad 29: Net-(A1-GPIO22) -> unconnected-(A1-GPIO22-Pad29)_1
- A1 pad 40: +5C -> unconnected-(A1-VBUS-Pad40)_1
- A1 pad 5: unconnected-(A1-GPIO3-Pad5) -> Net-(A1-GPIO3)
- C6 pad 1: unconnected-(C6-Pad1) -> GNDA
- D1 pad 1: Net-(A1-GPIO22) -> Net-(D1-A1)
- D1 pad 2: Net-(D1-K) -> GND
- D2 pad 1: Net-(D1-A2) -> Net-(D2-A1)
- D2 pad 2: Net-(D2-K) -> GND
- D2 pad 3: Net-(A1-GPIO22) -> Net-(D2-A2)
- R2 pad 2: Net-(D1-K) -> Net-(D2-A2)
- R3 pad 2: Net-(D2-K) -> Net-(D2-A1)
Routing:
- net unconnected-(A1-GPIO3-Pad5): track 52.2 -> 0.00 mm, vias 4 -> 0
- net Net-(A1-GPIO3): track 0.00 -> 52.2 mm, vias 0 -> 4

Commit message: KiCad
Parts:
- removed SW2: Select Waveform LFO2, Button_Switch_THT:SW_PUSH_6mm
- added R16: 100, Resistor_SMD:R_1206_3216Metric, F.Cu at (105.3, 43.7)
- SW1: value Select Waveform LFO1 -> Select Waveform LFO
- moved D1 60.0 mm to (104.2, 39.2), turned to 0 degrees
- moved D2 50.2 mm to (127.9, 37.1)
- moved SW1 18.0 mm to (141.2, 96.2)
Connections:
- A1 pad 33: GNDA -> GND
- A1 pad 4: unconnected-(A1-GPIO2-Pad4) -> Net-(A1-GPIO2)
- C2 pad 1: GNDA -> GND
- C3 pad 1: GNDA -> GND
- C4 pad 1: GNDA -> GND
- C6 pad 1: GNDA -> GND
- R13 pad 3: GNDA -> GND
- R14 pad 3: GNDA -> GND
- R15 pad 3: GNDA -> GND
- SW1 pad 2: Net-(A1-GPIO4) -> Net-(A1-GPIO2)
Routing:
- net GND: track 103.0 -> 209.8 mm, vias 6 -> 12
- net GNDA: track 106.8 -> 0.00 mm, vias 6 -> 0

Commit message: KiCad
Parts:
- removed R16, R17: 100, Resistor_SMD:R_1206_3216Metric
- added SW2: selectWaveForm, Button_Switch_THT:SW-MS-500X-3, F.Cu at (120.0, 94.0)
- A1: footprint RPI:Raspberry_Pi_Pico_SMT_THT_noDebugPort -> RPI_pico_Module:Raspberry_Pi_Pico_SMT_THT_noDebugPort
- D1: value LED_LFO2 -> LED LFO1; footprint LED_THT:LED_D3.0mm-3 -> LED_THT:LED_D3.0mm
- D2: value LED_LFO1 -> LED LFO2; footprint LED_THT:LED_D3.0mm-3 -> LED_THT:LED_D3.0mm
- SW1: value Select Waveform LFO -> LFO
- moved D1 61.8 mm to (143.4, 87.0), turned to 180 degrees
- moved D2 50.5 mm to (135.2, 87.0)
- moved R2 10.4 mm to (138.8, 88.4), turned to 90 degrees
- moved R3 6.53 mm to (130.7, 88.4), turned to 90 degrees
- moved R8 6.39 mm to (170.5, 88.4), turned to -90 degrees
- moved R7 6.27 mm to (152.5, 88.3), turned to -90 degrees
Connections:
- A1 pad 19: Net-(A1-GPIO14) -> unconnected-(A1-GPIO14-Pad19)
- A1 pad 20: Net-(A1-GPIO15) -> unconnected-(A1-GPIO15-Pad20)
- D1 pad 1: Net-(D1-A1) -> GND
- D1 pad 2: GND -> Net-(D1-A)
- D2 pad 1: Net-(D2-A1) -> GND
- D2 pad 2: GND -> Net-(D2-A)
- R2 pad 2: Net-(D2-A2) -> Net-(D1-A)
- R3 pad 2: Net-(D2-A1) -> Net-(D2-A)
Routing:
- net Net-(A1-GPIO4): track 50.6 -> 35.1 mm, vias 4 -> 2
- net Net-(A1-GPIO3): track 52.2 -> 37.0 mm, vias 4 -> 2

Commit message: KiCad MatrixLED und Bauteil für Echo
Parts:
- removed J3: Wave Out, Connector_PinSocket_2.54mm:PinSocket_1x02_P2.54mm_Vertical
- removed J4: Echo Out, Connector_PinSocket_2.54mm:PinSocket_1x02_P2.54mm_Vertical
- removed J5: Poti Echo Mix/Feedback, Connector_PinSocket_2.54mm:PinSocket_1x03_P2.54mm_Vertical
- removed J6: Poti Echo Freq, Connector_PinSocket_2.54mm:PinSocket_1x03_P2.54mm_Vertical
- removed J7: Echo Power, Connector_PinSocket_2.54mm:PinSocket_1x02_P2.54mm_Vertical
- added D10: LED WF_Tri, LED_THT:LED_D3.0mm, F.Cu at (121.3, 87.0)
- added D11: LED WF_Saw, LED_THT:LED_D3.0mm, F.Cu at (127.4, 87.0)
- added D12: ZMDxx, Diode_SMD:D_MiniMELF, B.Cu at (132.9, 53.6)
- added D8: LED WF_Squ, LED_THT:LED_D3.0mm, F.Cu at (115.2, 87.0)
- added U1: PT2399 Modul, PT2399_modul:PT2399_modul, F.Cu at (240.3, 15.6)
- SW1: value LFO -> LFO1/2
- SW2: value selectWaveForm -> Select LFO WaveForm; footprint Button_Switch_THT:SW-MS-500X-3 -> Button_Switch_THT:SW_PUSH_6mm
- moved SW6 16.1 mm to (53.8, 121.8)
- moved SW3 16.0 mm to (161.8, 121.8)
- moved SW4 16.0 mm to (125.8, 121.8)
- moved SW5 16.0 mm to (89.8, 121.8)
- moved C1 5.14 mm to (146.9, 68.3)
- moved SW2 3.95 mm to (123.2, 96.2), turned to 180 degrees
- moved D2 1.02 mm to (136.3, 87.0)
- moved D1 1.01 mm to (142.4, 87.0)
Connections:
- A1 pad 19: unconnected-(A1-GPIO14-Pad19) -> Net-(A1-GPIO14)
- A1 pad 20: unconnected-(A1-GPIO15-Pad20) -> Net-(A1-GPIO15)
- A1 pad 4: Net-(A1-GPIO2) -> unconnected-(A1-GPIO2-Pad4)
- A1 pad 5: Net-(A1-GPIO3) -> unconnected-(A1-GPIO3-Pad5)
- A1 pad 6: Net-(A1-GPIO4) -> unconnected-(A1-GPIO4-Pad6)
- D3 pad 1: GND -> Net-(A1-GPIO14)
- D4 pad 1: GND -> Net-(A1-GPIO13)
- D5 pad 1: GND -> Net-(A1-GPIO14)
- D5 pad 2: Net-(D5-A) -> Net-(D4-A)
- D6 pad 1: GND -> Net-(A1-GPIO15)
- D6 pad 2: Net-(D6-A) -> Net-(D4-A)
- D7 pad 1: GND -> Net-(A1-GPIO13)
- D7 pad 2: Net-(D7-A) -> Net-(D3-A)
- D9 pad 1: GND -> Net-(A1-GPIO15)
- D9 pad 2: Net-(D9-A) -> Net-(D3-A)
- R10 pad 1: Net-(D5-A) -> Net-(D3-A)
- R11 pad 1: Net-(D6-A) -> Net-(D10-A)
- SW1 pad 2: Net-(A1-GPIO2) -> Net-(A1-GPIO9)
- SW2 pad 1: Net-(A1-GPIO3) -> GND
- SW2 pad 2: GND -> Net-(A1-GPIO8)
Routing:
- net GND: track 209.8 -> 165.2 mm
- net unconnected-(A1-GPIO3-Pad5)_1: track 0.00 -> 37.0 mm, vias 0 -> 2
- net Net-(A1-GPIO3): track 37.0 -> 0.00 mm, vias 2 -> 0
- net unconnected-(A1-GPIO4-Pad6)_1: track 0.00 -> 35.1 mm, vias 0 -> 2
- net Net-(A1-GPIO4): track 35.1 -> 0.00 mm, vias 2 -> 0
- net +5C: track 116.3 -> 91.2 mm
- net Net-(U1-Freq_S): track 18.7 -> 0.00 mm
- net Net-(RV5-Pad1): track 18.6 -> 0.00 mm
- net Net-(RV5-Pad2): track 18.3 -> 0.00 mm
- net Net-(U1-Mix_G): track 18.3 -> 0.16 mm
- net Net-(A1-GPIO13): track 111.8 -> 123.1 mm
- net Net-(A1-GPIO15): track 0.00 -> 11.2 mm
- net Net-(U1-Mix_S): track 18.8 -> 10.7 mm
- net Net-(A1-GPIO18): track 19.0 -> 11.0 mm
- net Net-(U1-Mix_D): track 18.9 -> 11.0 mm
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Other:
- board size 142 x 67 mm -> 142 x 81 mm

Commit message: KiCad
Parts:
- added Q1: 2N7002, Package_TO_SOT_SMD:SOT-23, B.Cu at (64.9, 113.3)
- added Q2: 2N7002, Package_TO_SOT_SMD:SOT-23, B.Cu at (68.9, 113.3)
- added Q3: 2N7002, Package_TO_SOT_SMD:SOT-23, B.Cu at (73.0, 113.3)
- added Q4: 2N7002, Package_TO_SOT_SMD:SOT-23, B.Cu at (77.1, 113.3)
- added Q5: 2N7002, Package_TO_SOT_SMD:SOT-23, B.Cu at (81.1, 113.3)
- added Q6: 2N7002, Package_TO_SOT_SMD:SOT-23, B.Cu at (85.2, 113.3)
- added R16: 100, Resistor_SMD:R_1206_3216Metric, B.Cu at (79.1, 95.0)
- added R17: 100, Resistor_SMD:R_1206_3216Metric, B.Cu at (79.1, 100.1)
- added R18: 100, Resistor_SMD:R_1206_3216Metric, B.Cu at (79.1, 102.6)
- D1: value LED LFO1 -> LED LFO2
- D2: value LED LFO2 -> LED LFO1
- R12, R7, R8: value 100 -> 1k
- moved R12 93.7 mm to (79.1, 92.4)
- moved R8 91.5 mm to (79.1, 89.9), turned to 0 degrees
- moved R7 73.4 mm to (79.1, 87.4), turned to 0 degrees
- moved R11 38.1 mm to (112.6, 81.8), turned to 90 degrees
- moved R10 28.7 mm to (70.0, 108.9), turned to -90 degrees
- moved R1 20.9 mm to (90.8, 56.6)
- moved C5 9.86 mm to (69.7, 58.4), turned to 90 degrees
- moved R3 7.04 mm to (133.7, 82.0), turned to -90 degrees
- moved C6 6.65 mm to (53.7, 75.9), turned to 90 degrees
- moved R2 6.49 mm to (139.8, 82.0), turned to -90 degrees
- moved R9 5.40 mm to (65.9, 108.9), turned to -90 degrees
- moved C3 0.25 mm to (60.3, 85.1)
- moved C4 0.25 mm to (60.3, 75.9)
Connections:
- A1 pad 33: GND -> GNDA
- C2 pad 1: GND -> GNDA
- C3 pad 1: GND -> GNDA
- C4 pad 1: GND -> GNDA
- C6 pad 1: GND -> GNDA
- D10 pad 1: Net-(A1-GPIO14) -> Net-(D10-K)
- D11 pad 1: Net-(A1-GPIO15) -> Net-(D11-K)
- D3 pad 1: Net-(A1-GPIO14) -> Net-(D10-K)
- D4 pad 1: Net-(A1-GPIO13) -> Net-(D4-K)
- D5 pad 1: Net-(A1-GPIO14) -> Net-(D10-K)
- D6 pad 1: Net-(A1-GPIO15) -> Net-(D11-K)
- D7 pad 1: Net-(A1-GPIO13) -> Net-(D4-K)
- D8 pad 1: Net-(A1-GPIO13) -> Net-(D4-K)
- D9 pad 1: Net-(A1-GPIO15) -> Net-(D11-K)
- R10 pad 2: Net-(A1-GPIO11) -> Net-(Q2-S)
- R11 pad 2: Net-(A1-GPIO12) -> Net-(Q3-S)
- R12 pad 2: Net-(A1-GPIO13) -> Net-(A1-GPIO12)
- R13 pad 3: GND -> GNDA
- R14 pad 3: GND -> GNDA
- R15 pad 3: GND -> GNDA
- R7 pad 1: Net-(D3-A) -> Net-(Q1-G)
- R7 pad 2: Net-(A1-GPIO8) -> Net-(A1-GPIO10)
- R8 pad 2: Net-(A1-GPIO9) -> Net-(A1-GPIO11)
- R9 pad 2: Net-(A1-GPIO10) -> Net-(Q1-S)
Routing:
- net Net-(A1-GPIO21): track 139.0 -> 6.50 mm, vias 2 -> 0
- net GND: track 165.2 -> 34.0 mm, vias 12 -> 3
- net Net-(A1-GPIO13): track 123.1 -> 3.36 mm
- net Net-(D4-A): track 5.20 -> 92.5 mm
- net Net-(A1-GPIO20): track 87.2 -> 6.50 mm, vias 2 -> 0
- net +5C: track 91.2 -> 11.7 mm
- net Net-(A1-GPIO16): track 75.4 -> 0.00 mm, vias 1 -> 0
- net Net-(A1-GPIO17): track 75.4 -> 0.00 mm, vias 1 -> 0
- net Net-(A1-GPIO12): track 66.5 -> 3.36 mm
- net Net-(A1-GPIO11): track 57.3 -> 3.36 mm
- net Net-(A1-GPIO19): track 47.1 -> 6.50 mm, vias 2 -> 0
- net Net-(A1-GPIO10): track 42.4 -> 3.36 mm
- net unconnected-(A1-GPIO3-Pad5)_1 (its old number): track 37.0 -> 0.00 mm, vias 2 -> 0
- net Net-(Q1-G): track 0.00 -> 35.2 mm
- net unconnected-(A1-GPIO4-Pad6)_1 (its old number): track 35.1 -> 0.00 mm, vias 2 -> 0
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
Commit message: Kicad
Routing:
- net Net-(Q3-S): track 0.00 -> 67.4 mm, vias 0 -> 2
- net GND: track 34.0 -> 94.5 mm
- net Net-(D10-A): track 0.00 -> 3.77 mm
- net Net-(D2-A): track 0.00 -> 3.52 mm
- net Net-(D1-A): track 0.00 -> 3.52 mm
- net GNDA: track 33.9 -> 33.0 mm
- net Net-(Q2-G): track 29.0 -> 28.5 mm
- net Net-(Q1-G): track 35.2 -> 34.6 mm

Commit message: Kicad
Parts:
- moved R11 6.14 mm to (109.6, 87.1), turned to -90 degrees
Routing:
- net Net-(A1-GPIO7): track 0.00 -> 94.4 mm
- net Net-(A1-GPIO6): track 0.00 -> 80.3 mm, vias 0 -> 2
- net Net-(D11-K): track 0.00 -> 79.9 mm, vias 0 -> 2
- net Net-(D4-K): track 25.6 -> 80.6 mm, vias 0 -> 2
- net Net-(A1-GPIO8): track 0.00 -> 44.5 mm
- net Net-(D10-K): track 16.3 -> 59.6 mm
- net Net-(A1-GPIO5): track 0.00 -> 20.6 mm
- net Net-(A1-GPIO27_ADC1): track 3.31 -> 20.2 mm
- net Net-(Q3-S): track 67.4 -> 51.2 mm
- net GNDA: track 33.0 -> 46.2 mm
