File: KiCad/VCO_RPIpico.kicad_pcb (KiCad board)
At the start: 2 copper layers, 138 x 83 mm, 81 parts, among them J1 AudioJack3_Ground, J2 Power Jack, SW1 LFO1/2, SW2 Select LFO WaveForm, SW3 Fire4, SW4 Fire3, SW5 Fire2, SW6 Fire1, SW7 Shift2/Save, SW8 Shift1 / Select Bank, U2 PT2399, U3 L7805

Commit message: Kicad: Muting control added
Routing:
- net GND: vias 47 -> 34
